Commit message: Simulación estable. Cámara simulada funcional con parámetros ov5647. Nodo de detección de pelota calibrado con menos del 5% de error.

File: prueba2_ws/src/c_ros_sim/urdf/c_ros_bot.urdf (robot description, URDF)
Before this commit: robot c_ros_bot, 6 links, 5 joints
Links:
- added link camera_link, mass 0.01; visual box size=0.02 0.06 0.04
Joints:
- added joint camera_joint: type fixed, parent base_link, child camera_link, origin xyz=0 0.075 0.125 rpy=0 0.3490 1.5708
- joint caster_wheel2_joint: origin xyz=0 0.10 0.015 rpy=0 0 0 -> xyz=0 0.065 -0.008 rpy=0 0 0
- joint caster_wheel_joint: origin xyz=0 0.10 0.015 rpy=0 0 0 -> xyz=0 -0.065 -0.008 rpy=0 0 0
- joint left_wheel_joint: origin xyz=0.10 0 0.034 rpy=0 0 1.5708 -> xyz=0.069 -0.005 0.012 rpy=0 0 1.5708
- joint right_wheel_joint: origin xyz=-0.10 0 0.034 rpy=0 0 1.5708 -> xyz=-0.069 -0.005 0.012 rpy=0 0 1.5708
