Commit message: se agregaron diferentes launch ademas del lidar de la simulacion

File: simulation_ws/src/c_ros_sim/urdf/c_ros_bot.urdf (robot description, URDF)
Before this commit: robot c_ros_bot, 7 links, 6 joints
Links:
- added link lidar_link, mass 0.1; collision cylinder length=0.04 radius=0.03; visual cylinder length=0.03 radius=0.03
- link base_link: geometry collision box size=0.25 0.15 0.05; visual mesh filename=package://c_ros_sim/meshes/Futbot3.0.stl scale=0.001 0.001 0.001
Joints:
- added joint lidar_joint: type fixed, parent base_link, child lidar_link, origin xyz=0.0 0 0.075 rpy=0 0 0
